File: stm_32_v2.0.sch (EAGLE design)
At the start: 76 parts, among them IC1 ESP-07S, J1 6_PIN_SERIAL_CABLEPTH, J2 6_PIN_SERIAL_CABLEPTH, T1 BC847, T2 BC847, T3 BC847

Commit message: updated schematic
Parts:
- added C12, C13: 22nF, adafruit:C-USC0805
- added U1: AMS1117-3.3, AMS1117-3.3:AMS1117-3.3
Connections:
- new net VCC5V: C12.2, C13.2, U1.ADJ/GND
- net VCC: now also C12.1, C13.1, U1.VIN, U1.VOUT
Changed lines of the file:
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@@
 <part name="SUPPLY28" library="supply2" library_urn="urn:adsk.eagle:library:372" deviceset="GND" device=""/>
 <part name="P+15" library="supply1" library_urn="urn:adsk.eagle:library:371" deviceset="VCC" device="" value="VCC 3.3"/>
+<part name="U1" library="AMS1117-3.3" deviceset="AMS1117-3.3" device=""/>
+<part name="C12" library="adafruit" library_urn="urn:adsk.eagle:library:420" deviceset="C-US" device="C0805" package3d_urn="urn:adsk.eagle:package:6240337/1" value="22nF"/>
+<part name="C13" library="adafruit" library_urn="urn:adsk.eagle:library:420" deviceset="C-US" device="C0805" package3d_urn="urn:adsk.eagle:package:6240337/1" value="22nF"/>
+<part name="SUPPLY29" library="supply2" library_urn="urn:adsk.eagle:library:372" deviceset="GND" device=""/>
+<part name="VCC5V3" library="supply1" library_urn="urn:adsk.eagle:library:371" deviceset="VCC" device="" value="VCC5V"/>
+<part name="P+16" library="supply1" library_urn="urn:adsk.eagle:library:371" deviceset="VCC" device="" value="VCC 3.3"/>
 </parts>
 <sheets>
@@
 </instance>
 <instance part="P+4" gate="VCC" x="86.36" y="170.18" smashed="yes" rot="R270">
-<attribute name="VALUE" x="73.66" y="170.18" size="1.778" layer="96"/>
+<attribute name="VALUE" x="78.74" y="167.64" size="1.778" layer="96"/>
 </instance>
 <instance part="P+5" gate="VCC" x="96.52" y="195.58" smashed="yes">
@@
 <instance part="P+15" gate="VCC" x="129.54" y="22.86" smashed="yes">
 <attribute name="VALUE" x="127" y="20.32" size="1.778" layer="96" rot="R90"/>
+</instance>
+<instance part="U1" gate="G$1" x="50.8" y="147.32" smashed="yes" rot="R180">
+<attribute name="NAME" x="60.9766" y="141.722859375" size="2.54415" layer="95" rot="R180"/>
+<attribute name="VALUE" x="60.9692" y="155.455359375" size="2.5423" layer="96" rot="R180"/>
+</instance>
+<instance part="C12" gate="G$1" x="30.48" y="144.78" smashed="yes" rot="R270">
+<attribute name="VALUE" x="26.289" y="143.764" size="1.778" layer="96" rot="R270"/>
+</instance>
+<instance part="C13" gate="G$1" x="68.58" y="149.86" smashed="yes" rot="R180">
+<attribute name="VALUE" x="67.564" y="154.051" size="1.778" layer="96" rot="R180"/>
+</instance>
+<instance part="SUPPLY29" gate="GND" x="20.32" y="149.86" smashed="yes" rot="R270">
+<attribute name="VALUE" x="17.145" y="151.765" size="1.778" layer="96" rot="R270"/>
+</instance>
+<instance part="VCC5V3" gate="VCC" x="68.58" y="139.7" smashed="yes" rot="R180">
+<attribute name="VALUE" x="71.12" y="144.78" size="1.778" layer="96" rot="R270"/>
+</instance>
+<instance part="P+16" gate="VCC" x="35.56" y="139.7" smashed="yes" rot="R180">
+<attribute name="VALUE" x="38.1" y="142.24" size="1.778" layer="96" rot="R270"/>
 </instance>
 </instances>
@@
 <wire x1="129.54" y1="20.32" x2="129.54" y2="15.24" width="0.1524" layer="91"/>
 </segment>
+<segment>
+<pinref part="C13" gate="G$1" pin="1"/>
+<wire x1="68.58" y1="144.78" x2="68.58" y2="147.32" width="0.1524" layer="91"/>
+<pinref part="U1" gate="G$1" pin="VIN"/>
+<wire x1="66.04" y1="144.78" x2="68.58" y2="144.78" width="0.1524" layer="91"/>
+<pinref part="VCC5V3" gate="VCC" pin="VCC"/>
+<wire x1="68.58" y1="142.24" x2="68.58" y2="144.78" width="0.1524" layer="91"/>
+<junction x="68.58" y="144.78"/>
+</segment>
+<segment>
+<pinref part="C12" gate="G$1" pin="1"/>
+<pinref part="U1" gate="G$1" pin="VOUT"/>
+<wire x1="33.02" y1="144.78" x2="35.56" y2="144.78" width="0.1524" layer="91"/>
+<pinref part="P+16" gate="VCC" pin="VCC"/>
+<wire x1="35.56" y1="142.24" x2="35.56" y2="144.78" width="0.1524" layer="91"/>
+<junction x="35.56" y="144.78"/>
+</segment>
 </net>
 <net name="N$21" class="0">
@@
 </segment>
 </net>
+<net name="VCC5V" class="0">
+<segment>
+<pinref part="C12" gate="G$1" pin="2"/>
+<pinref part="U1" gate="G$1" pin="ADJ/GND"/>
+<wire x1="25.4" y1="144.78" x2="25.4" y2="149.86" width="0.1524" layer="91"/>
+<wire x1="25.4" y1="149.86" x2="30.48" y2="149.86" width="0.1524" layer="91"/>
+<pinref part="SUPPLY29" gate="GND" pin="GND"/>
+<wire x1="30.48" y1="149.86" x2="35.56" y2="149.86" width="0.1524" layer="91"/>
+<wire x1="22.86" y1="149.86" x2="25.4" y2="149.86" width="0.1524" layer="91"/>
+<junction x="25.4" y="149.86"/>
+<pinref part="C13" gate="G$1" pin="2"/>
+<wire x1="68.58" y1="154.94" x2="68.58" y2="157.48" width="0.1524" layer="91"/>
+<wire x1="68.58" y1="157.48" x2="30.48" y2="157.48" width="0.1524" layer="91"/>
+<wire x1="30.48" y1="157.48" x2="30.48" y2="149.86" width="0.1524" layer="91"/>
+<junction x="30.48" y="149.86"/>
+</segment>
+</net>
